Commit message: Save current project progress

File: src/robot_package/urdf/robot.urdf (robot description, URDF)
Before this commit: robot esp32_robot, 5 links, 4 joints
Links:
- added link laser_frame; visual cylinder length=0.04 radius=0.035
Joints:
- added joint laser_joint: type fixed, parent base_link, child laser_frame, origin xyz=0.05 0.0 0.10 rpy=0 0 0
